File: Test_Project.kicad_sch (KiCad schematic)
At the start: 67 parts, among them J2 Conn_01x02, J3 Conn_01x03, J4 Conn_01x03, J5 Conn_01x04, J6 Conn_01x04, Q1 NTTFS5C454NLTAG, Q2 NTTFS5C454NLTAG, Q3 NTTFS5C454NLTAG, Q4 NTTFS5C454NLTAG, Q5 Q_NMOS_DSG, U1 STM32L081KZTx, U2 MIC2132YML

Commit message: Started PCB layout
Parts:
- removed J4: Conn_01x03, Connector_PinHeader_2.54mm:PinHeader_1x03_P2.54mm_Vertical, symbol Library:Conn_01x03
- added C33: 22uF, Capacitor_SMD:C_0805_2012Metric_Pad1.18x1.45mm_HandSolder, symbol Library:C_Small_US
- added F1: 0678L9300-02, Test_Project_Lib:Fuse - 0678L9300-02, symbol Device:Fuse
- added J4: Conn_01x04, Connector_PinHeader_2.54mm:PinHeader_1x04_P2.54mm_Vertical, symbol Library:Conn_01x04
- added R20: 3.3k, Resistor_SMD:R_0805_2012Metric_Pad1.20x1.40mm_HandSolder, symbol Library:R_Small
- C18: value ?uF -> 100nF
- L1, L2: footprint (none) -> Test_Project_Lib:SRP1265A
- Q1, Q2, Q3, Q4: footprint (none) -> Test_Project_Lib:NTTFS5C454NLTAG
- Q5: value Q_NMOS_DSG -> BSS138-7-F; footprint (none) -> Test_Project_Lib:BSS138-7-F
- R1: value 100k -> 1M
- U3: value ~ -> AP2127N-3.3TRG1
Connections:
- net 12V: now also F1.1
- net Boot0: now also C33.1, R20.2
- net USART_RX: now also J4.3 (Pin_3)
- net USART_TX: now also J4.2 (Pin_2)
- net VDD_3V3: now also J4.1 (Pin_1)
- net Vin: now also F1.2
- net GND: now reaches C2.2, C3.2, C4.2, C5.2
- net GND: now also C1.2, C10.2, C11.2, C12.2, C13.2, C15.2, C16.2, C18.2, C19.2, C20.2, C21.2, C22.2, C23.2, C24.2, C25.2, C26.2, C27.2, C28.2, C29.2, C30.2, C31.2, C32.2, C6.1, C7.1, J1.3, J2.2 (Pin_2), J3.3 (Pin_3), J5.4 (Pin_4), J6.4 (Pin_4), Q2.2 (S), Q4.2 (S), R1.2, R14.1, R16.1, R17.1, R4.1, R5.1, U1.16 (VSS), U1.32 (VSS), U2.1 (CSN2), U2.10 (AGND), U2.20 (PGND), U2.29 (GFB), U2.3 (CSN1), U2.33 (PAD), U3.1 (GND), C33.2, J4.4 (Pin_4)
- net Vout_ADC: now reaches C32.1, R15.1, R17.2
- net Vout_ADC: now also U1.15 (PB1)
- net Bootloader_On_Reset: now reaches U1.6 (PA0)
- net Bootloader_On_Reset: now also R20.1
- net Vin_ADC: now reaches U1.9 (PA3)
- net Vin_ADC: now also C31.1, R16.2, R8.1
Other:
- note added: "ADC_IN3"
- note added: "ADC_IN9"
- note removed: "*Verify LDO footprint before going for it"
- moved on the sheet: C1, C31, C32, J5, J6, R15, R16, R17, R8

Commit message: Removed the 12V jack, added another 0.1" header in parallel so more current can be achieved if there are issues. Did most of the PCB layout. Updated some footprints
Parts:
- removed J1: ~, Connector_BarrelJack:BarrelJack_GCT_DCJ200-10-A_Horizontal, symbol Library:Barrel_Jack_Switch_Pin3Ring
- added J1: Conn_01x02, Connector_PinHeader_2.54mm:PinHeader_1x02_P2.54mm_Vertical, symbol Library:Conn_01x02
- added J7: Conn_01x04, Connector_PinHeader_2.54mm:PinHeader_1x04_P2.54mm_Vertical, symbol Library:Conn_01x04
- F1: symbol Device:Fuse -> Library:Fuse
Connections:
- net 12V: now also J1.1 (Pin_1)
- net GND: now also R11.2, J1.2 (Pin_2), J7.4 (Pin_4)
- net SWCLK: now also J7.3 (Pin_3)
- net SWDIO: now also J7.2 (Pin_2)
- net Vin_ADC: now also U1.15 (PB1); no longer U1.9 (PA3)
- net Vout_ADC: now also U1.9 (PA3); no longer U1.15 (PB1)
- net nRST: now also J7.1 (Pin_1)
Other:
- moved on the sheet: J2

Commit message: Finished up routing nets and pouring polygons. Needs final ground pours and review before ordering.
Connections:
- net VDD_5V: now also R2.2; no longer R2.1
- net at U2.26 (PG): now also R2.1; no longer R2.2
Other:
- moved on the sheet: R2
Changed lines of the file:
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@@
 	(symbol
 		(lib_id "Library:R_Small")
-		(at 123.19 97.79 90)
+		(at 123.19 97.79 270)
+		(mirror x)
 		(unit 1)
 		(exclude_from_sim no)
@@
 		(on_board yes)
 		(dnp no)
-		(fields_autoplaced yes)
 		(property "Reference" "R2"
 			(at 123.19 92.71 90)

Commit message: Finished up layout and added some mounting holes.
Parts:
- C1, C10, C12, C14, C17, C18, C2, C28, C3, C4, C7, C9: Digikey_PN (none) -> 1276-1006-1-ND; Part Number (none) -> CL10B104KA8NNNC
- C11, C13, C29, C30, C31, C32, C5, C8: Digikey_PN (none) -> 1276-1184-1-ND; Part Number (none) -> CL10B105KA8NNNC
- C15, C16, C21, C22, C23, C24, C25, C26, C33: Digikey_PN (none) -> 1276-CL21A226MAYNNNECT-ND; Part Number (none) -> CL21A226MAYNNNE
- C19, C20: Digikey_PN (none) -> 1276-1044-1-ND; Part Number (none) -> CL10A475KP8NNNC
- C27: Digikey_PN (none) -> 399-6613-ND; Part Number (none) -> EST107M025AE3AA
- C6: Digikey_PN (none) -> 1276-1008-1-ND; Part Number (none) -> CL10C101JB8NNNC
- F1: Digikey_PN (none) -> 5923-0678L9300-02CT-ND; Part Number (none) -> 0678L9300-02
- J1, J2, J3, J4, J5, J6, J7: Digikey_PN (none) -> x; Part Number (none) -> x
- L1, L2: Digikey_PN (none) -> SRP1265A-2R2MCT-ND; Part Number (none) -> SRP1265A-2R2M
- Q1, Q2, Q3, Q4: Digikey_PN (none) -> NTTFS5C454NLTAGOSCT-ND; Part Number (none) -> NTTFS5C454NLTAG
- Q5: Digikey_PN (none) -> BSS138-FDICT-ND; Part Number (none) -> BSS138-7-F
- R1: Digikey_PN (none) -> 541-5248-1-ND; Part Number (none) -> CRCW06031M00FKEAC
- R10, R11, R12, R6, R8: value 100k -> 100kΩ; Digikey_PN (none) -> 541-100KHCT-ND; Part Number (none) -> CRCW0603100KFKEA
- R13: Digikey_PN (none) -> 541-2.20HHCT-ND; Part Number (none) -> CRCW06032R20FKEA
- R14, R20, R7: value 3.3k -> 3.3kΩ; Digikey_PN (none) -> 541-CRCW06033K30JNEACCT-ND; Part Number (none) -> CRCW06033K30JNEAC
- R15, R18, R19, R4, R5: Digikey_PN (none) -> 541-25.5KHCT-ND; Part Number (none) -> CRCW060325K5FKEA
- R16, R17, R2, R3: value 10k -> 10kΩ; Digikey_PN (none) -> 541-10.0KHCT-ND; Part Number (none) -> CRCW060310K0FKEA
- R9: Digikey_PN (none) -> 541-10.0KHCT-ND; Part Number (none) -> CRCW060310K0FKEA
- U1: value STM32L081KZTx -> STM32L081KZT6; Digikey_PN (none) -> 497-16832-ND; Part Number (none) -> STM32L081KZTx
- U2: Digikey_PN (none) -> 150-MIC2132YML-TRCT-ND; Part Number (none) -> MIC2132YML
- U3: Digikey_PN (none) -> AP2127N-3.3TRG1DICT-ND; Part Number (none) -> AP2127N-3.3TRG1
Other:
- note added: "Current MOSFETs may have too low Vgs threshhold..."
- note added: "I_{LIM}=30A per phase"
- note added: "In this configuration, when R_{ILIM} is set to: 100k -> 7A phase limit 92k -> 10A phase limit 75k -> 15A phase limit 45k -> 24A phase limit"
- note added: "R_{DSON} assumed to be 8m"
- note removed: "*Verify MOSFET footprint before going for it"
- note removed: "I_{LIM}=12A per phase"
- note removed: "R_{DSON} assumed to be 20m"
- note removed: "Read datasheet on using capacitors that are not low ESR..."

Commit message: Daily commit. Working through test points and DRC checks.
Parts:
- renumbered C29 to C1, C5 to C10, C8 to C11, C9 to C12, C7 to C13, C6 to C14, C18 to C15, C19 to C16, C20 to C17, C17 to C18, C14 to C19, C4 to C2, C21 to C20, C15 to C21, C16 to C23, C12 to C24, C10 to C25, C13 to C26, C11 to C27, C24 to C28, C23 to C29, C1 to C3, C26 to C30, C25 to C31, C27 to C32, C32 to C33, C2 to C4, C28 to C5, C33 to C6, C30 to C7, C3 to C8, C31 to C9, J2 to J1, J1 to J2, J4 to J3, J5 to J4, J6 to J5, J7 to J6, J3 to J7, R8 to R1, R4 to R10, R10 to R11, R20 to R12, R2 to R13, R3 to R14, R12 to R15, R13 to R16, R18 to R17, R19 to R18, R15 to R19, R16 to R2, R17 to R20, R1 to R3, R9 to R4, R7 to R5, R14 to R6, R6 to R7, R11 to R8, R5 to R9, U3 to U1, U1 to U2, U2 to U3
